File: board-game-counter/board/board.brd (EAGLE design)
At the start: 71.1 x 64.8 mm, 42 parts, among them IC1 TINY13-20PU, IC2 74HCT595N, IC3 74HCT595N, T1 A42, T2 A42, T3 A42, T4 A42, T5 S9013

Commit message: board-game-counter updated
Parts:
- R19: value 1.5k -> 1k
Changed lines of the file:
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@@
 <element name="5.1V" library="diode" library_urn="urn:adsk.eagle:library:210" package="DO41Z10" package3d_urn="urn:adsk.eagle:package:43341/1" value="1N4728" x="40.64" y="46.99" rot="R180"/>
 <element name="C4" library="resistor" library_urn="urn:adsk.eagle:library:348" package="E3,5-8" package3d_urn="urn:adsk.eagle:package:25842/1" value="1000uf" x="40.64" y="38.1" rot="R180"/>
-<element name="R19" library="resistor" library_urn="urn:adsk.eagle:library:348" package="0207/2V" package3d_urn="urn:adsk.eagle:package:25941/1" value="1.5k" x="38.1" y="24.13"/>
+<element name="R19" library="resistor" library_urn="urn:adsk.eagle:library:348" package="0207/2V" package3d_urn="urn:adsk.eagle:package:25941/1" value="1k" x="38.1" y="24.13"/>
 <element name="U$3" library="mgvc" package="TRANS" value="TRANS" x="43.18" y="13.97"/>
 <element name="VCC-RAW" library="wirepad" library_urn="urn:adsk.eagle:library:412" package="2,54/0,8" package3d_urn="urn:adsk.eagle:package:30838/1" value="" x="39.37" y="13.97"/>
